File: RPi-HwAB-1.kicad_sch (KiCad schematic)
At the start: 11 parts, among them J1 GPIO, J2 Hirose_FH12-16S, J3 TC2030, J4 Conn_ARM_SWD_TagConnect_TC203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, U1 XC7A35T-FGG484, U2 CAT24C256, U3 ADP5054

Commit message: file restructuring
redefined naming scheme for schematic files (fpga-num) etc.
Other:
- sheet FPGA 2: file fpga-15.kicad_sch -> fpga-2.kicad_sch
- sheet FPGA 3: file fpga-mgt.kicad_sch -> fpga-3.kicad_sch
Changed lines of the file:
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@@
 			)
 		)
-		(property "Sheetfile" "fpga-mgt.kicad_sch"
+		(property "Sheetfile" "fpga-3.kicad_sch"
 			(at 83.82 142.8246 0)
 			(effects
@@
 	)
 	(sheet
-		(at -2.54 -31.75)
+		(at 67.31 -31.75)
 		(size 24.13 21.59)
 		(exclude_from_sim no)
@@
 		)
 		(property "Sheetname" "FPGA 2"
-			(at -2.54 -32.4616 0)
+			(at 67.31 -32.4616 0)
 			(effects
 				(font
@@
 			)
 		)
-		(property "Sheetfile" "fpga-15.kicad_sch"
-			(at -2.54 -9.5754 0)
+		(property "Sheetfile" "fpga-2.kicad_sch"
+			(at 67.31 -9.5754 0)
 			(effects
 				(font
@@
 	)
 	(sheet
-		(at -41.91 -15.24)
+		(at 40.64 -29.21)
 		(size 19.05 19.05)
 		(exclude_from_sim no)
@@
 		)
 		(property "Sheetname" "FPGA 1"
-			(at -41.91 -15.9516 0)
+			(at 40.64 -29.9216 0)
 			(effects
 				(font
@@
 		)
 		(property "Sheetfile" "fpga-1.kicad_sch"
-			(at -41.91 4.3946 0)
+			(at 40.64 -9.5754 0)
 			(effects
 				(font
