File: fpga-pwr.kicad_sch (KiCad schematic)
At the start: 3 parts

Commit message: file restructuring
redefined naming scheme for schematic files (fpga-num) etc.
Other:
- note added: "Power sequencing:"
Changed lines of the file:
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@@
 	(generator_version "9.0")
 	(paper "A4")
+	(text "Power sequencing: \n"
+		(exclude_from_sim no)
+		(at 234.95 90.17 0)
+		(effects
+			(font
+				(size 1.27 1.27)
+			)
+		)
+	)
 	(junction
 		(at 100.33 113.03)
