File: pcb/sequencing.kicad_sch (KiCad schematic)
At the start: 8 parts, among them U10 TXS0102YZP, U9 LM3880

Commit message: defined memory pinouts
Parts:
- renumbered C103 to C16, C104 to C17, C102 to C18, R26 to R22, R27 to R23, R28 to R24, U9 to U3, U10 to U4

Commit message: power restructuring
Parts:
- renumbered C18 to C10, C16 to C8, C17 to C9, R22 to R18, R23 to R19, R24 to R20
Changed lines of the file:
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@@
+	)
+	(junction
+		(at 116.84 90.17)
+		(diameter 0)
+		(color 0 0 0 0)
 	)
 	(junction
@@
 	)
 	(junction
-		(at 118.11 90.17)
-		(diameter 0)
-		(color 0 0 0 0)
-	)
-	(junction
 		(at 149.86 67.31)
 		(diameter 0)
@@
 	(wire
 		(pts
-			(xy 114.3 90.17) (xy 118.11 90.17)
+			(xy 114.3 90.17) (xy 116.84 90.17)
 		)
 		(stroke
@@
 	(wire
 		(pts
+			(xy 116.84 128.27) (xy 118.11 128.27)
+		)
+		(stroke
+			(width 0)
+			(type default)
+		)
+	)
+	(wire
+		(pts
 			(xy 90.17 67.31) (xy 114.3 67.31)
 		)
@@
 	(wire
 		(pts
+			(xy 116.84 90.17) (xy 118.11 90.17)
+		)
+		(stroke
+			(width 0)
+			(type default)
+		)
+	)
+	(wire
+		(pts
 			(xy 166.37 82.55) (xy 166.37 119.38)
 		)
@@
 	(wire
 		(pts
-			(xy 118.11 128.27) (xy 118.11 133.35)
+			(xy 116.84 128.27) (xy 116.84 133.35)
 		)
 		(stroke
@@
 	(wire
 		(pts
-			(xy 118.11 92.71) (xy 118.11 90.17)
+			(xy 116.84 92.71) (xy 116.84 90.17)
 		)
 		(stroke
@@
 		(on_board yes)
 		(dnp no)
-		(property "Reference" "C18"
+		(property "Reference" "C10"
 			(at 153.67 125.7299 0)
 			(effects
@@
 		(instances
 			(project "RPi-HwAB-1"
-				(path "/e63e39d7-6ac0-4ffd-8aa3-1841a4541b55/f9ebb56c-78c7-42ac-bc19-ccbf788f5318/39d2a084-247a-4d14-8064-0b32c2eb111e"
-					(reference "C18")
+				(path "/e63e39d7-6ac0-4ffd-8aa3-1841a4541b55/f9ebb56c-78c7-42ac-bc19-ccbf788f5318/3b0633e7-b2c4-49de-84a6-497b0545e0f9"
+					(reference "C10")
 					(unit 1)
 				)
@@
 		(instances
 			(project "RPi-HwAB-1"
-				(path "/e63e39d7-6ac0-4ffd-8aa3-1841a4541b55/f9ebb56c-78c7-42ac-bc19-ccbf788f5318/39d2a084-247a-4d14-8064-0b32c2eb111e"
+				(path "/e63e39d7-6ac0-4ffd-8aa3-1841a4541b55/f9ebb56c-78c7-42ac-bc19-ccbf788f5318/3b0633e7-b2c4-49de-84a6-497b0545e0f9"
 					(reference "U4")
 					(unit 1)
@@
 		(dnp no)
 		(fields_autoplaced yes)
-		(property "Reference" "#PWR017"
+		(property "Reference" "#PWR013"
 			(at 149.86 139.7 0)
 			(effects
@@
 		(instances
 			(project "RPi-HwAB-1"
-				(path "/e63e39d7-6ac0-4ffd-8aa3-1841a4541b55/f9ebb56c-78c7-42ac-bc19-ccbf788f5318/39d2a084-247a-4d14-8064-0b32c2eb111e"
-					(reference "#PWR017")
+				(path "/e63e39d7-6ac0-4ffd-8aa3-1841a4541b55/f9ebb56c-78c7-42ac-bc19-ccbf788f5318/3b0633e7-b2c4-49de-84a6-497b0545e0f9"
+					(reference "#PWR013")
 					(unit 1)
 				)
@@
 		(on_board yes)
 		(dnp no)
-		(property "Reference" "C16"
+		(property "Reference" "C8"
 			(at 105.41 125.7299 0)
 			(effects
@@
 		(instances
 			(project "RPi-HwAB-1"
-				(path "/e63e39d7-6ac0-4ffd-8aa3-1841a4541b55/f9ebb56c-78c7-42ac-bc19-ccbf788f5318/39d2a084-247a-4d14-8064-0b32c2eb111e"
-					(reference "C16")
+				(path "/e63e39d7-6ac0-4ffd-8aa3-1841a4541b55/f9ebb56c-78c7-42ac-bc19-ccbf788f5318/3b0633e7-b2c4-49de-84a6-497b0545e0f9"
+					(reference "C8")
 					(unit 1)
 				)
@@
 		(dnp no)
 		(fields_autoplaced yes)
-		(property "Reference" "#PWR014"
+		(property "Reference" "#PWR010"
 			(at 109.22 139.7 0)
 			(effects
@@
 		(instances
 			(project "RPi-HwAB-1"
-				(path "/e63e39d7-6ac0-4ffd-8aa3-1841a4541b55/f9ebb56c-78c7-42ac-bc19-ccbf788f5318/39d2a084-247a-4d14-8064-0b32c2eb111e"
-					(reference "#PWR014")
+				(path "/e63e39d7-6ac0-4ffd-8aa3-1841a4541b55/f9ebb56c-78c7-42ac-bc19-ccbf788f5318/3b0633e7-b2c4-49de-84a6-497b0545e0f9"
+					(reference "#PWR010")
 					(unit 1)
 				)
@@
 	(symbol
 		(lib_id "library:GND")
-		(at 118.11 133.35 0)
+		(at 116.84 133.35 0)
 		(unit 1)
 		(exclude_from_sim no)
@@
 		(dnp no)
 		(fields_autoplaced yes)
-		(property "Reference" "#PWR016"
-			(at 118.11 139.7 0)
+		(property "Reference" "#PWR012"
+			(at 116.84 139.7 0)
 			(effects
 				(font
@@
 		)
 		(property "Value" "GND"
-			(at 118.11 138.43 0)
+			(at 116.84 138.43 0)
 			(effects
 				(font
@@
 		)
 		(property "Footprint" ""
-			(at 118.11 133.35 0)
+			(at 116.84 133.35 0)
 			(effects
 				(font
@@
 		)
 		(property "Datasheet" ""
-			(at 118.11 133.35 0)
+			(at 116.84 133.35 0)
 			(effects
 				(font
@@
 		)
 		(property "Description" "Power symbol creates a global label with name \"GND\" , ground"
-			(at 118.11 133.35 0)
+			(at 116.84 133.35 0)
 			(effects
 				(font
@@
 		(instances
 			(project "RPi-HwAB-1"
-				(path "/e63e39d7-6ac0-4ffd-8aa3-1841a4541b55/f9ebb56c-78c7-42ac-bc19-ccbf788f5318/39d2a084-247a-4d14-8064-0b32c2eb111e"
-					(reference "#PWR016")
+				(path "/e63e39d7-6ac0-4ffd-8aa3-1841a4541b55/f9ebb56c-78c7-42ac-bc19-ccbf788f5318/3b0633e7-b2c4-49de-84a6-497b0545e0f9"
+					(reference "#PWR012")
 					(unit 1)
 				)
@@
 		(on_board yes)
 		(dnp no)
-		(property "Reference" "C17"
+		(property "Reference" "C9"
 			(at 110.49 85.0899 0)
 			(effects
@@
 		(instances
 			(project "RPi-HwAB-1"
-				(path "/e63e39d7-6ac0-4ffd-8aa3-1841a4541b55/f9ebb56c-78c7-42ac-bc19-ccbf788f5318/39d2a084-247a-4d14-8064-0b32c2eb111e"
-					(reference "C17")
+				(path "/e63e39d7-6ac0-4ffd-8aa3-1841a4541b55/f9ebb56c-78c7-42ac-bc19-ccbf788f5318/3b0633e7-b2c4-49de-84a6-497b0545e0f9"
+					(reference "C9")
 					(unit 1)
 				)
@@
 		(dnp no)
 		(fields_autoplaced yes)
-		(property "Reference" "R23"
+		(property "Reference" "R19"
 			(at 189.23 74.9299 0)
 			(effects
@@
 		(instances
 			(project "RPi-HwAB-1"
-				(path "/e63e39d7-6ac0-4ffd-8aa3-1841a4541b55/f9ebb56c-78c7-42ac-bc19-ccbf788f5318/39d2a084-247a-4d14-8064-0b32c2eb111e"
-					(reference "R23")
+				(path "/e63e39d7-6ac0-4ffd-8aa3-1841a4541b55/f9ebb56c-78c7-42ac-bc19-ccbf788f5318/3b0633e7-b2c4-49de-84a6-497b0545e0f9"
+					(reference "R19")
 					(unit 1)
 				)
@@
 	(symbol
 		(lib_id "library:GND")
-		(at 118.11 92.71 0)
+		(at 116.84 92.71 0)
 		(unit 1)
 		(exclude_from_sim no)
@@
 		(dnp no)
 		(fields_autoplaced yes)
-		(property "Reference" "#PWR015"
-			(at 118.11 99.06 0)
+		(property "Reference" "#PWR011"
+			(at 116.84 99.06 0)
 			(effects
 				(font
@@
 		)
 		(property "Value" "GND"
-			(at 118.11 97.79 0)
+			(at 116.84 97.79 0)
 			(effects
 				(font
@@
 		)
 		(property "Footprint" ""
-			(at 118.11 92.71 0)
+			(at 116.84 92.71 0)
 			(effects
 				(font
@@
 		)
 		(property "Datasheet" ""
-			(at 118.11 92.71 0)
+			(at 116.84 92.71 0)
 			(effects
 				(font
@@
 		)
 		(property "Description" "Power symbol creates a global label with name \"GND\" , ground"
-			(at 118.11 92.71 0)
+			(at 116.84 92.71 0)
 			(effects
 				(font
@@
 		(instances
 			(project "RPi-HwAB-1"
-				(path "/e63e39d7-6ac0-4ffd-8aa3-1841a4541b55/f9ebb56c-78c7-42ac-bc19-ccbf788f5318/39d2a084-247a-4d14-8064-0b32c2eb111e"
-					(reference "#PWR015")
+				(path "/e63e39d7-6ac0-4ffd-8aa3-1841a4541b55/f9ebb56c-78c7-42ac-bc19-ccbf788f5318/3b0633e7-b2c4-49de-84a6-497b0545e0f9"
+					(reference "#PWR011")
 					(unit 1)
 				)
@@
 		(dnp no)
 		(fields_autoplaced yes)
-		(property "Reference" "R24"
+		(property "Reference" "R20"
 			(at 199.39 74.9299 0)
 			(effects
@@
 		(instances
 			(project "RPi-HwAB-1"
-				(path "/e63e39d7-6ac0-4ffd-8aa3-1841a4541b55/f9ebb56c-78c7-42ac-bc19-ccbf788f5318/39d2a084-247a-4d14-8064-0b32c2eb111e"
-					(reference "R24")
+				(path "/e63e39d7-6ac0-4ffd-8aa3-1841a4541b55/f9ebb56c-78c7-42ac-bc19-ccbf788f5318/3b0633e7-b2c4-49de-84a6-497b0545e0f9"
+					(reference "R20")
 					(unit 1)
 				)
@@
 		(instances
 			(project "RPi-HwAB-1"
-				(path "/e63e39d7-6ac0-4ffd-8aa3-1841a4541b55/f9ebb56c-78c7-42ac-bc19-ccbf788f5318/39d2a084-247a-4d14-8064-0b32c2eb111e"
+				(path "/e63e39d7-6ac0-4ffd-8aa3-1841a4541b55/f9ebb56c-78c7-42ac-bc19-ccbf788f5318/3b0633e7-b2c4-49de-84a6-497b0545e0f9"
 					(reference "U3")
 					(unit 1)
@@
 		(dnp no)
 		(fields_autoplaced yes)
-		(property "Reference" "R22"
+		(property "Reference" "R18"
 			(at 179.07 74.9299 0)
 			(effects
@@
 		(instances
 			(project "RPi-HwAB-1"
-				(path "/e63e39d7-6ac0-4ffd-8aa3-1841a4541b55/f9ebb56c-78c7-42ac-bc19-ccbf788f5318/39d2a084-247a-4d14-8064-0b32c2eb111e"
-					(reference "R22")
+				(path "/e63e39d7-6ac0-4ffd-8aa3-1841a4541b55/f9ebb56c-78c7-42ac-bc19-ccbf788f5318/3b0633e7-b2c4-49de-84a6-497b0545e0f9"
+					(reference "R18")
 					(unit 1)
 				)
