File: pcb/connectors.kicad_sch (KiCad schematic)
At the start: 5 parts, among them J1 GPIO, J2 Hirose_FH12-16S, J3 TC2030

Commit message: decoupling
Changed lines of the file:
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@@
 		(members "CLK_P" "CLK_N" "F2P_P" "F2P_N" "P2F_P" "P2F_N")
+	)
+	(bus_alias "PCIEsb"
+		(members "PWR_EN" "DET_WAKE" "CLKREQ_N" "RST_B")
 	)
 	(rectangle
@@
 	)
 	(label "PCIE.F2P_P"
-		(at 209.55 116.84 0)
+		(at 208.28 116.84 0)
 		(effects
 			(font
@@
 	)
 	(label "PCIE.CLKREQ_N"
-		(at 209.55 137.16 0)
+		(at 208.28 137.16 0)
 		(effects
 			(font
@@
 	)
 	(label "PCIE.RST_B"
-		(at 209.55 139.7 0)
+		(at 208.28 139.7 0)
 		(effects
 			(font
@@
 	)
 	(label "PCIE.DET_WAKE"
-		(at 209.55 134.62 0)
+		(at 208.28 134.62 0)
 		(effects
 			(font
@@
 	)
 	(label "PCIE.P2F_N"
-		(at 209.55 127 0)
+		(at 208.28 127 0)
 		(effects
 			(font
@@
 	)
 	(label "PCIE.PWR_EN"
-		(at 209.55 132.08 0)
+		(at 208.28 132.08 0)
 		(effects
 			(font
@@
 	)
 	(label "PCIE.P2F_P"
-		(at 209.55 124.46 0)
+		(at 208.28 124.46 0)
 		(effects
 			(font
@@
 	)
 	(label "PCIE.CLK_N"
-		(at 209.55 111.76 0)
+		(at 208.28 111.76 0)
 		(effects
 			(font
@@
 	)
 	(label "PCIE.CLK_P"
-		(at 209.55 109.22 0)
+		(at 208.28 109.22 0)
 		(effects
 			(font
@@
 	)
 	(label "PCIE.F2P_N"
-		(at 209.55 119.38 0)
-		(effects
-			(font
+		(at 208.28 119.38 0)
+		(effects
+			(font
