File: pcb/connectors.kicad_sch (KiCad schematic)
At the start: 5 parts, among them J1 GPIO, J2 Hirose_FH12-16S, J3 TC2030

Commit message: bom
Parts:
- J1: Manufacturer (none) -> Samtec Inc.; Manufacturer Product Number (none) -> SSQ-120-03-G-D; Part Description (none) -> CONN RCPT 40POS 0.1 GOLD PCB
- J2: Manufacturer (none) -> Hirose Electric Co Ltd; Manufacturer Product Number (none) -> FH12-16S-1SH(55); Part Description (none) -> CONN FFC FPC BOTTOM 16POS 1MM RA
- R29: renamed from R27; footprint library:R_0402_1005Metric -> Resistor_SMD:R_0402_1005Metric; Manufacturer YAGEO -> Vishay Dale; Manufacturer Product Number RC0402FR-07100KL -> CRCW0402100KFKED; Part Description (none) -> RES 100K OHM 1% 1/16W 0402
- R30: renamed from R28; Manufacturer (none) -> Vishay Dale; Manufacturer Product Number (none) -> CRCW04022K20FKED; Part Description (none) -> RES 2.2K OHM 1% 1/16W 0402
Connections:
- net 3V3: no longer J1.1 (Pin_1), J1.17 (Pin_17), R30.1
- new net 3V3_RPi: J1.1 (Pin_1), J1.17 (Pin_17), R30.1
Changed lines of the file:
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@@
 		)
 	)
-	(label "3V3"
+	(label "3V3_RPi"
 		(at 53.34 63.5 0)
 		(effects
@@
 		)
 	)
-	(label "3V3"
+	(label "3V3_RPi"
 		(at 251.46 115.57 180)
 		(effects
@@
 		)
 	)
-	(hierarchical_label "3V3"
+	(hierarchical_label "3V3_RPi"
 		(shape output)
 		(at 50.8 63.5 180)
@@
 		(on_board yes)
 		(dnp no)
-		(property "Reference" "#PWR045"
+		(property "Reference" "#PWR063"
 			(at 101.6 129.54 0)
 			(effects
@@
 			(project "RPi-HwAB-1"
 				(path "/e63e39d7-6ac0-4ffd-8aa3-1841a4541b55/6418cef5-c0d2-4573-8432-9553c4202f1e"
-					(reference "#PWR045")
+					(reference "#PWR063")
 					(unit 1)
 				)
@@
 		(on_board yes)
 		(dnp no)
-		(property "Reference" "#PWR044"
+		(property "Reference" "#PWR062"
 			(at 83.82 129.54 0)
 			(effects
@@
 			(project "RPi-HwAB-1"
 				(path "/e63e39d7-6ac0-4ffd-8aa3-1841a4541b55/6418cef5-c0d2-4573-8432-9553c4202f1e"
-					(reference "#PWR044")
+					(reference "#PWR062")
 					(unit 1)
 				)
@@
 		)
 		(property "Description" "Generic connector, double row, 02x20, odd/even pin numbering scheme (row 1 odd numbers, row 2 even numbers), script generated (kicad-library-utils/schlib/autogen/connector/)"
+			(at 91.44 93.98 0)
+			(effects
+				(font
+					(size 1.27 1.27)
+				)
+				(hide yes)
+			)
+		)
+		(property "Manufacturer" "Samtec Inc."
+			(at 91.44 93.98 0)
+			(effects
+				(font
+					(size 1.27 1.27)
+				)
+				(hide yes)
+			)
+		)
+		(property "Manufacturer Product Number" "SSQ-120-03-G-D"
+			(at 91.44 93.98 0)
+			(effects
+				(font
+					(size 1.27 1.27)
+				)
+				(hide yes)
+			)
+		)
+		(property "Part Description" "CONN RCPT 40POS 0.1 GOLD PCB"
 			(at 91.44 93.98 0)
 			(effects
@@
 		(on_board yes)
 		(dnp no)
-		(property "Reference" "#PWR046"
+		(property "Reference" "#PWR064"
 			(at 200.66 158.75 0)
 			(effects
@@
 			(project "RPi-HwAB-1"
 				(path "/e63e39d7-6ac0-4ffd-8aa3-1841a4541b55/6418cef5-c0d2-4573-8432-9553c4202f1e"
-					(reference "#PWR046")
+					(reference "#PWR064")
 					(unit 1)
 				)
@@
 		(dnp no)
 		(fields_autoplaced yes)
-		(property "Reference" "R28"
+		(property "Reference" "R30"
 			(at 241.3 121.9199 0)
 			(effects
@@
 		)
 		(property "Description" "Resistor, US symbol"
+			(at 238.76 123.19 0)
+			(effects
+				(font
+					(size 1.27 1.27)
+				)
+				(hide yes)
+			)
+		)
+		(property "Manufacturer" "Vishay Dale"
+			(at 238.76 123.19 0)
+			(effects
+				(font
+					(size 1.27 1.27)
+				)
+				(hide yes)
+			)
+		)
+		(property "Manufacturer Product Number" "CRCW04022K20FKED"
+			(at 238.76 123.19 0)
+			(effects
+				(font
+					(size 1.27 1.27)
+				)
+				(hide yes)
+			)
+		)
+		(property "Part Description" "RES 2.2K OHM 1% 1/16W 0402"
 			(at 238.76 123.19 0)
 			(effects
@@
 			(project ""
 				(path "/e63e39d7-6ac0-4ffd-8aa3-1841a4541b55/6418cef5-c0d2-4573-8432-9553c4202f1e"
-					(reference "R28")
+					(reference "R30")
 					(unit 1)
 				)
@@
 			)
 		)
+		(property "Manufacturer" "Hirose Electric Co Ltd"
+			(at 191.77 121.92 0)
+			(effects
+				(font
+					(size 1.27 1.27)
+				)
+				(hide yes)
+			)
+		)
+		(property "Manufacturer Product Number" "FH12-16S-1SH(55)"
+			(at 191.77 121.92 0)
+			(effects
+				(font
+					(size 1.27 1.27)
+				)
+				(hide yes)
+			)
+		)
+		(property "Part Description" "CONN FFC FPC BOTTOM 16POS 1MM RA"
+			(at 191.77 121.92 0)
+			(effects
+				(font
+					(size 1.27 1.27)
+				)
+				(hide yes)
+			)
+		)
 		(pin "16"
 		)
@@
 		(on_board yes)
 		(dnp no)
-		(property "Reference" "#PWR048"
+		(property "Reference" "#PWR066"
 			(at 226.06 158.75 0)
 			(effects
@@
 			(project "RPi-HwAB-1"
 				(path "/e63e39d7-6ac0-4ffd-8aa3-1841a4541b55/6418cef5-c0d2-4573-8432-9553c4202f1e"
-					(reference "#PWR048")
+					(reference "#PWR066")
 					(unit 1)
 				)
@@
 		(on_board yes)
 		(dnp no)
-		(property "Reference" "#PWR049"
+		(property "Reference" "#PWR067"
 			(at 233.68 158.75 0)
 			(effects
@@
 			(project "RPi-HwAB-1"
 				(path "/e63e39d7-6ac0-4ffd-8aa3-1841a4541b55/6418cef5-c0d2-4573-8432-9553c4202f1e"
-					(reference "#PWR049")
+					(reference "#PWR067")
 					(unit 1)
 				)
@@
 		(dnp no)
 		(fields_autoplaced yes)
-		(property "Reference" "R27"
+		(property "Reference" "R29"
 			(at 236.22 144.7799 0)
 			(effects
@@
 			)
 		)
-		(property "Footprint" "library:R_0402_1005Metric"
+		(property "Footprint" "Resistor_SMD:R_0402_1005Metric"
 			(at 232.664 145.796 90)
 			(effects
@@
 			)
 		)
-		(property "Manufacturer" "YAGEO"
+		(property "Manufacturer" "Vishay Dale"
 			(at 233.68 146.05 0)
 			(effects
@@
 			)
 		)
-		(property "Manufacturer Product Number" "RC0402FR-07100KL"
+		(property "Manufacturer Product Number" "CRCW0402100KFKED"
 			(at 233.68 146.05 90)
+			(effects
+				(font
+					(size 1.27 1.27)
+				)
+				(hide yes)
+			)
+		)
+		(property "Part Description" "RES 100K OHM 1% 1/16W 0402"
+			(at 233.68 146.05 0)
 			(effects
 				(font
@@
 			(project "RPi-HwAB-1"
 				(path "/e63e39d7-6ac0-4ffd-8aa3-1841a4541b55/6418cef5-c0d2-4573-8432-9553c4202f1e"
-					(reference "R27")
+					(reference "R29")
 					(unit 1)
 				)
@@
 		(dnp no)
 		(fields_autoplaced yes)
-		(property "Reference" "#PWR047"
+		(property "Reference" "#PWR065"
 			(at 209.55 71.12 0)
 			(effects
@@
 			(project "RPi-HwAB-1"
 				(path "/e63e39d7-6ac0-4ffd-8aa3-1841a4541b55/6418cef5-c0d2-4573-8432-9553c4202f1e"
-					(reference "#PWR047")
+					(reference "#PWR065")
 					(unit 1)
 				)

Commit message: added mig ddr pinout constraints
Parts:
- renumbered R30 to R29, R29 to R30
Connections:
- net 3V3 is gone; now on net 3V3_RPi: J3.1
- net 3V3_RPi: no longer R29.1
- new net 3V3_FD: R29.1
Changed lines of the file:
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@@
 	(wire
 		(pts
-			(xy 191.77 40.64) (xy 200.66 40.64)
+			(xy 193.04 40.64) (xy 205.74 40.64)
 		)
 		(stroke
@@
 	(wire
 		(pts
-			(xy 238.76 115.57) (xy 251.46 115.57)
-		)
-		(stroke
-			(width 0.254)
-			(type default)
-			(color 0 0 255 1)
+			(xy 238.76 114.3) (xy 246.38 114.3)
+		)
+		(stroke
+			(width 0)
+			(type default)
 		)
 	)
@@
 	(wire
 		(pts
-			(xy 238.76 115.57) (xy 238.76 119.38)
-		)
-		(stroke
-			(width 0.254)
-			(type default)
-			(color 0 0 255 1)
+			(xy 238.76 114.3) (xy 238.76 119.38)
+		)
+		(stroke
+			(width 0)
+			(type default)
 		)
 	)
@@
 	(wire
 		(pts
-			(xy 200.66 40.64) (xy 200.66 58.42)
+			(xy 205.74 40.64) (xy 205.74 58.42)
 		)
 		(stroke
@@
 	(wire
 		(pts
-			(xy 200.66 96.52) (xy 218.44 96.52)
+			(xy 200.66 96.52) (xy 220.98 96.52)
 		)
 		(stroke
@@
 	(wire
 		(pts
-			(xy 200.66 58.42) (xy 210.82 58.42)
+			(xy 205.74 58.42) (xy 210.82 58.42)
 		)
 		(stroke
@@
 		)
 	)
-	(label "3V3_RPi"
-		(at 251.46 115.57 180)
-		(effects
-			(font
-				(size 1.27 1.27)
-			)
-			(justify right bottom)
-		)
-	)
 	(label "PCIE.RST_B"
 		(at 208.28 139.7 0)
@@
 		)
 	)
-	(label "3V3"
-		(at 191.77 40.64 0)
+	(label "3V3_RPi"
+		(at 195.58 40.64 0)
 		(effects
 			(font
@@
 		)
 	)
+	(hierarchical_label "3V3_RPi"
+		(shape output)
+		(at 193.04 40.64 180)
+		(effects
+			(font
+				(size 1.27 1.27)
+			)
+			(justify right)
+		)
+	)
 	(hierarchical_label "PCIE.PWR_EN"
 		(shape output)
@@
 		)
 	)
+	(hierarchical_label "5V0"
+		(shape output)
+		(at 220.98 96.52 0)
+		(effects
+			(font
+				(size 1.27 1.27)
+			)
+			(justify left)
+		)
+	)
 	(hierarchical_label "{JTAG}"
 		(shape bidirectional)
 		(at 132.08 109.22 0)
+		(effects
+			(font
+				(size 1.27 1.27)
+			)
+			(justify left)
+		)
+	)
+	(hierarchical_label "3V3_FD"
+		(shape input)
+		(at 246.38 114.3 0)
 		(effects
 			(font
@@
 		(on_board yes)
 		(dnp no)
-		(property "Reference" "#PWR063"
+		(property "Reference" "#PWR060"
 			(at 101.6 129.54 0)
 			(effects
@@
 			(project "RPi-HwAB-1"
 				(path "/e63e39d7-6ac0-4ffd-8aa3-1841a4541b55/6418cef5-c0d2-4573-8432-9553c4202f1e"
-					(reference "#PWR063")
+					(reference "#PWR060")
 					(unit 1)
 				)
@@
 		(on_board yes)
 		(dnp no)
-		(property "Reference" "#PWR062"
+		(property "Reference" "#PWR059"
 			(at 83.82 129.54 0)
 			(effects
@@
 			(project "RPi-HwAB-1"
 				(path "/e63e39d7-6ac0-4ffd-8aa3-1841a4541b55/6418cef5-c0d2-4573-8432-9553c4202f1e"
-					(reference "#PWR062")
+					(reference "#PWR059")
 					(unit 1)
 				)
@@
 		(on_board yes)
 		(dnp no)
-		(property "Reference" "#PWR064"
+		(property "Reference" "#PWR061"
 			(at 200.66 158.75 0)
 			(effects
@@
 			(project "RPi-HwAB-1"
 				(path "/e63e39d7-6ac0-4ffd-8aa3-1841a4541b55/6418cef5-c0d2-4573-8432-9553c4202f1e"
-					(reference "#PWR064")
+					(reference "#PWR061")
 					(unit 1)
 				)
@@
 		(dnp no)
 		(fields_autoplaced yes)
-		(property "Reference" "R30"
+		(property "Reference" "R29"
 			(at 241.3 121.9199 0)
 			(effects
@@
 			(project ""
 				(path "/e63e39d7-6ac0-4ffd-8aa3-1841a4541b55/6418cef5-c0d2-4573-8432-9553c4202f1e"
-					(reference "R30")
+					(reference "R29")
 					(unit 1)
 				)
@@
 		(on_board yes)
 		(dnp no)
-		(property "Reference" "#PWR066"
+		(property "Reference" "#PWR062"
 			(at 226.06 158.75 0)
 			(effects
@@
 			(project "RPi-HwAB-1"
 				(path "/e63e39d7-6ac0-4ffd-8aa3-1841a4541b55/6418cef5-c0d2-4573-8432-9553c4202f1e"
-					(reference "#PWR066")
+					(reference "#PWR062")
 					(unit 1)
 				)
@@
 		(on_board yes)
 		(dnp no)
-		(property "Reference" "#PWR067"
+		(property "Reference" "#PWR063"
 			(at 233.68 158.75 0)
 			(effects
@@
 			(project "RPi-HwAB-1"
 				(path "/e63e39d7-6ac0-4ffd-8aa3-1841a4541b55/6418cef5-c0d2-4573-8432-9553c4202f1e"
-					(reference "#PWR067")
+					(reference "#PWR063")
 					(unit 1)
 				)
@@
 		(dnp no)
 		(fields_autoplaced yes)
-		(property "Reference" "R29"
+		(property "Reference" "R30"
 			(at 236.22 144.7799 0)
 			(effects
@@
 			(project "RPi-HwAB-1"
 				(path "/e63e39d7-6ac0-4ffd-8aa3-1841a4541b55/6418cef5-c0d2-4573-8432-9553c4202f1e"
-					(reference "R29")
+					(reference "R30")
 					(unit 1)
 				)
@@
 		(dnp no)
 		(fields_autoplaced yes)
-		(property "Reference" "#PWR065"
+		(property "Reference" "#PWR058"
 			(at 209.55 71.12 0)
 			(effects
@@
 			(project "RPi-HwAB-1"
 				(path "/e63e39d7-6ac0-4ffd-8aa3-1841a4541b55/6418cef5-c0d2-4573-8432-9553c4202f1e"
-					(reference "#PWR065")
+					(reference "#PWR058")
 					(unit 1)
 				)

Commit message: restructured power, power plane layout
Parts:
- renumbered J3 to J1, J1 to J2, J2 to J3, R29 to R23, R30 to R24
Changed lines of the file:
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@@
-		)
-	)
-	(rule_area
-		(polyline
-			(pts
-				(xy 208.28 105.41) (xy 205.74 107.95) (xy 205.74 125.73) (xy 208.28 128.27) (xy 223.52 128.27) (xy 226.06 125.73)
-				(xy 226.06 107.95) (xy 223.52 105.41)
-			)
-			(stroke
-				(width 0.2032)
-				(type dash)
-			)
-			(fill
-				(type none)
-			)
-		)
-	)
-	(netclass_flag ""
-		(length 2.54)
-		(shape round)
-		(at 209.55 105.41 0)
-		(fields_autoplaced yes)
-		(effects
-			(font
-				(size 1.27 1.27)
-			)
-			(justify left bottom)
-		)
-		(property "Netclass" "Differential"
-			(at 210.439 102.87 0)
-			(effects
-				(font
-					(size 1.27 1.27)
-				)
-				(justify left)
-			)
-		)
-		(property "Component Class" "90 ohm"
-			(at 210.439 104.521 0)
-			(effects
-				(font
-					(size 1.27 1.27)
-					(italic yes)
-				)
-				(justify left)
-			)
 		)
 	)
@@
 		(on_board yes)
 		(dnp no)
-		(property "Reference" "#PWR060"
+		(property "Reference" "#PWR054"
 			(at 101.6 129.54 0)
 			(effects
@@
 			(project "RPi-HwAB-1"
 				(path "/e63e39d7-6ac0-4ffd-8aa3-1841a4541b55/6418cef5-c0d2-4573-8432-9553c4202f1e"
-					(reference "#PWR060")
+					(reference "#PWR054")
 					(unit 1)
 				)
@@
 		(on_board yes)
 		(dnp no)
-		(property "Reference" "#PWR059"
+		(property "Reference" "#PWR053"
 			(at 83.82 129.54 0)
 			(effects
@@
 			(project "RPi-HwAB-1"
 				(path "/e63e39d7-6ac0-4ffd-8aa3-1841a4541b55/6418cef5-c0d2-4573-8432-9553c4202f1e"
-					(reference "#PWR059")
+					(reference "#PWR053")
 					(unit 1)
 				)
@@
 		(on_board yes)
 		(dnp no)
-		(property "Reference" "J1"
+		(property "Reference" "J2"
 			(at 92.71 65.6398 0)
 			(effects
@@
 			(project "RPi-HwAB-1"
 				(path "/e63e39d7-6ac0-4ffd-8aa3-1841a4541b55/6418cef5-c0d2-4573-8432-9553c4202f1e"
-					(reference "J1")
+					(reference "J2")
 					(unit 1)
 				)
@@
 		(dnp no)
 		(fields_autoplaced yes)
-		(property "Reference" "#FLG07"
+		(property "Reference" "#FLG02"
 			(at 111.76 61.595 0)
 			(effects
@@
 			(project "RPi-HwAB-1"
 				(path "/e63e39d7-6ac0-4ffd-8aa3-1841a4541b55/6418cef5-c0d2-4573-8432-9553c4202f1e"
-					(reference "#FLG07")
+					(reference "#FLG02")
 					(unit 1)
 				)
@@
 		(on_board yes)
 		(dnp no)
-		(property "Reference" "#PWR061"
+		(property "Reference" "#PWR055"
 			(at 200.66 158.75 0)
 			(effects
@@
 			(project "RPi-HwAB-1"
 				(path "/e63e39d7-6ac0-4ffd-8aa3-1841a4541b55/6418cef5-c0d2-4573-8432-9553c4202f1e"
-					(reference "#PWR061")
+					(reference "#PWR055")
 					(unit 1)
 				)
@@
 		(dnp no)
 		(fields_autoplaced yes)
-		(property "Reference" "#FLG06"
+		(property "Reference" "#FLG01"
 			(at 71.12 61.595 0)
 			(effects
@@
 			(project ""
 				(path "/e63e39d7-6ac0-4ffd-8aa3-1841a4541b55/6418cef5-c0d2-4573-8432-9553c4202f1e"
-					(reference "#FLG06")
+					(reference "#FLG01")
 					(unit 1)
 				)
@@
 		(dnp no)
 		(fields_autoplaced yes)
-		(property "Reference" "R29"
+		(property "Reference" "R23"
 			(at 241.3 121.9199 0)
 			(effects
@@
 			(project ""
 				(path "/e63e39d7-6ac0-4ffd-8aa3-1841a4541b55/6418cef5-c0d2-4573-8432-9553c4202f1e"
-					(reference "R29")
+					(reference "R23")
 					(unit 1)
 				)
@@
 		(on_board yes)
 		(dnp no)
-		(property "Reference" "J2"
+		(property "Reference" "J3"
 			(at 193.04 99.06 0)
 			(effects
@@
 			(project "RPi-HwAB-1"
 				(path "/e63e39d7-6ac0-4ffd-8aa3-1841a4541b55/6418cef5-c0d2-4573-8432-9553c4202f1e"
-					(reference "J2")
+					(reference "J3")
 					(unit 1)
 				)
@@
 		(on_board yes)
 		(dnp no)
-		(property "Reference" "#PWR062"
+		(property "Reference" "#PWR056"
 			(at 226.06 158.75 0)
 			(effects
@@
 			(project "RPi-HwAB-1"
 				(path "/e63e39d7-6ac0-4ffd-8aa3-1841a4541b55/6418cef5-c0d2-4573-8432-9553c4202f1e"
-					(reference "#PWR062")
+					(reference "#PWR056")
 					(unit 1)
 				)
@@
 		(on_board yes)
 		(dnp no)
-		(property "Reference" "#PWR063"
+		(property "Reference" "#PWR057"
 			(at 233.68 158.75 0)
 			(effects
@@
 			(project "RPi-HwAB-1"
 				(path "/e63e39d7-6ac0-4ffd-8aa3-1841a4541b55/6418cef5-c0d2-4573-8432-9553c4202f1e"
-					(reference "#PWR063")
+					(reference "#PWR057")
 					(unit 1)
 				)
@@
 		(dnp no)
 		(fields_autoplaced yes)
-		(property "Reference" "J3"
+		(property "Reference" "J1"
 			(at 219.71 48.26 0)
 			(effects
@@
 			(project "RPi-HwAB-1"
 				(path "/e63e39d7-6ac0-4ffd-8aa3-1841a4541b55/6418cef5-c0d2-4573-8432-9553c4202f1e"
-					(reference "J3")
+					(reference "J1")
 					(unit 1)
 				)
@@
 		(dnp no)
 		(fields_autoplaced yes)
-		(property "Reference" "R30"
+		(property "Reference" "R24"
 			(at 236.22 144.7799 0)
 			(effects
@@
 			(project "RPi-HwAB-1"
 				(path "/e63e39d7-6ac0-4ffd-8aa3-1841a4541b55/6418cef5-c0d2-4573-8432-9553c4202f1e"
-					(reference "R30")
+					(reference "R24")
 					(unit 1)
 				)
@@
 		(dnp no)
 		(fields_autoplaced yes)
-		(property "Reference" "#PWR058"
+		(property "Reference" "#PWR052"
 			(at 209.55 71.12 0)
 			(effects
@@
 			(project "RPi-HwAB-1"
 				(path "/e63e39d7-6ac0-4ffd-8aa3-1841a4541b55/6418cef5-c0d2-4573-8432-9553c4202f1e"
-					(reference "#PWR058")
-					(unit 1)
-				)
+					(reference "#PWR052")
+					(unit 1)
+				)

Commit message: dogbone for ddr
Parts:
- added C1: 0.1uF, Capacitor_SMD:C_0402_1005Metric, symbol library:C_Small
- added JP1: ID_WP, Jumper:SolderJumper-2_P1.3mm_Open_Pad1.0x1.5mm, symbol library:SolderJumper_2_Open
- added R1, R2: 3.9k, Resistor_SMD:R_0402_1005Metric, symbol library:R_US
- added R25, R26, R27, R28, R29, R30: 100 1%, Resistor_SMD:R_0402_1005Metric, symbol library:R_US
- added U1: CAT24C256, Package_DFN_QFN:DFN-8-1EP_3x2mm_P0.5mm_EP1.7x1.4mm, symbol library:CAT24C256
Connections:
- net 3V3_FD: now also J1.1; no longer R23.1
- net 3V3_RPi: now also R23.1, C1.1, JP1.2 (B), R1.1, R2.1, U1.8 (VCC); no longer J1.1
- net DONE: now also R30.1; no longer J2.40 (Pin_40)
- net GND: now also C1.2, U1.4 (GND)
- net ID_SCL: now also R2.2, U1.6 (SCL)
- net ID_SDA: now also R1.2, U1.5 (SDA)
- net PROG_B: now also R29.1; no longer J2.38 (Pin_38)
- net TCK: now also R25.1; no longer J2.33 (Pin_33)
- net TDI: now also R27.1; no longer J2.37 (Pin_37)
- net TDO: now also R28.1; no longer J2.36 (Pin_36)
- net TMS: now also R26.1; no longer J2.35 (Pin_35)
- new net: JP1.1 (A), U1.7 (WP)
- new net DONE_RPi: J2.40 (Pin_40), R30.2
- new net PROG_B_RPi: J2.38 (Pin_38), R29.2
- new net TCK_RPi: J2.33 (Pin_33), R25.2
- new net TDI_RPi: J2.37 (Pin_37), R27.2
- new net TDO_RPi: J2.36 (Pin_36), R28.2
- new net TMS_RPi: J2.35 (Pin_35), R26.2
- no-connect marks 0 -> 3
Other:
- note added: "ID_SD and ID_SC PINS: These pins are reserved for HAT ID EEPROM. At boot time this I2C interface will be interrogated to look for an EEPROM that identifes the attached board and allows automagic setup of the GPIOs (and optionally, Linux drivers). Bridging JP1 enables write protection. DO NOT USE these pins for anything other than attaching an I2C ID EEPROM. Leave unconnected if ID EEPROM not requ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"
- moved on the sheet: J2

Commit message: ported to nightly, finished ddr routing yay!!!!!!! pcb/v1.0 almost complete!
Parts:
- removed R29, R30: 100 1%, Resistor_SMD:R_0402_1005Metric, symbol library:R_US
Connections:
- net DONE_RPi is gone; now on net TDO_RPi: J2.40 (Pin_40)
- net PROG_B_RPi is gone; now on net TDI_RPi: J2.38 (Pin_38)
- net TCK_RPi: now also J2.37 (Pin_37); no longer J2.33 (Pin_33)
- net TDI_RPi: no longer J2.37 (Pin_37)
- net TDO_RPi: no longer J2.36 (Pin_36)
- net TMS_RPi: now also J2.36 (Pin_36); no longer J2.35 (Pin_35)
