File: pcb/fpga-3.kicad_sch (KiCad schematic)
At the start: 13 parts, among them U7 XC7A100T-FGG484, Y1 SiT9365AI-2B2-33E200.000000

Commit message: restructured power, power plane layout
Parts:
- R16: renamed from R31; Part Description (none) -> RES SMD 100 OHM 1% 1/5W 0402
- renumbered C29 to C28, C30 to C29, C31 to C30, C32 to C31, C33 to C32, C34 to C33, C35 to C34, C36 to C35, R23 to R17, R24 to R18, U7 to U4
Changed lines of the file:
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@@
 		(dnp no)
 		(fields_autoplaced yes)
-		(property "Reference" "U7"
+		(property "Reference" "U4"
 			(at 147.32 17.78 0)
 			(effects
@@
 			(project "RPi-HwAB-1"
 				(path "/e63e39d7-6ac0-4ffd-8aa3-1841a4541b55/59d21473-a004-4514-8090-fd93db818925/143e814b-c088-43b0-8f2f-ada8c438e494"
-					(reference "U7")
+					(reference "U4")
 					(unit 6)
 				)
@@
 		(on_board yes)
 		(dnp no)
-		(property "Reference" "C31"
+		(property "Reference" "C30"
 			(at 219.71 138.43 0)
 			(effects
@@
 			(project "RPi-HwAB-1"
 				(path "/e63e39d7-6ac0-4ffd-8aa3-1841a4541b55/59d21473-a004-4514-8090-fd93db818925/143e814b-c088-43b0-8f2f-ada8c438e494"
-					(reference "C31")
+					(reference "C30")
 					(unit 1)
 				)
@@
 		(dnp no)
 		(fields_autoplaced yes)
-		(property "Reference" "#PWR029"
+		(property "Reference" "#PWR025"
 			(at 256.54 156.21 0)
 			(effects
@@
 			(project "RPi-HwAB-1"
 				(path "/e63e39d7-6ac0-4ffd-8aa3-1841a4541b55/59d21473-a004-4514-8090-fd93db818925/143e814b-c088-43b0-8f2f-ada8c438e494"
-					(reference "#PWR029")
+					(reference "#PWR025")
 					(unit 1)
 				)
@@
 		(dnp no)
 		(fields_autoplaced yes)
-		(property "Reference" "U7"
+		(property "Reference" "U4"
 			(at 35.56 17.78 0)
 			(effects
@@
 			(project "RPi-HwAB-1"
 				(path "/e63e39d7-6ac0-4ffd-8aa3-1841a4541b55/59d21473-a004-4514-8090-fd93db818925/143e814b-c088-43b0-8f2f-ada8c438e494"
-					(reference "U7")
+					(reference "U4")
 					(unit 5)
 				)
@@
 		(dnp no)
 		(fields_autoplaced yes)
-		(property "Reference" "R23"
+		(property "Reference" "R17"
 			(at 121.92 104.1399 0)
 			(effects
@@
 			(project "RPi-HwAB-1"
 				(path "/e63e39d7-6ac0-4ffd-8aa3-1841a4541b55/59d21473-a004-4514-8090-fd93db818925/143e814b-c088-43b0-8f2f-ada8c438e494"
-					(reference "R23")
+					(reference "R17")
 					(unit 1)
 				)
@@
 		(dnp no)
 		(fields_autoplaced yes)
-		(property "Reference" "R31"
+		(property "Reference" "R16"
 			(at 107.95 97.79 90)
 			(effects
@@
 			)
 		)
+		(property "Part Description" "RES SMD 100 OHM 1% 1/5W 0402"
+			(at 107.95 104.14 90)
+			(effects
+				(font
+					(size 1.27 1.27)
+				)
+				(hide yes)
+			)
+		)
 		(pin "2"
 		)
@@
 			(project ""
 				(path "/e63e39d7-6ac0-4ffd-8aa3-1841a4541b55/59d21473-a004-4514-8090-fd93db818925/143e814b-c088-43b0-8f2f-ada8c438e494"
-					(reference "R31")
+					(reference "R16")
 					(unit 1)
 				)
@@
 		(dnp no)
 		(fields_autoplaced yes)
-		(property "Reference" "R24"
+		(property "Reference" "R18"
 			(at 121.92 116.8399 0)
 			(effects
@@
 			(project "RPi-HwAB-1"
 				(path "/e63e39d7-6ac0-4ffd-8aa3-1841a4541b55/59d21473-a004-4514-8090-fd93db818925/143e814b-c088-43b0-8f2f-ada8c438e494"
-					(reference "R24")
+					(reference "R18")
 					(unit 1)
 				)
@@
 		(on_board yes)
 		(dnp no)
-		(property "Reference" "C36"
+		(property "Reference" "C35"
 			(at 257.81 138.43 0)
 			(effects
@@
 			(project "RPi-HwAB-1"
 				(path "/e63e39d7-6ac0-4ffd-8aa3-1841a4541b55/59d21473-a004-4514-8090-fd93db818925/143e814b-c088-43b0-8f2f-ada8c438e494"
-					(reference "C36")
+					(reference "C35")
 					(unit 1)
 				)
@@
 		(dnp no)
 		(fields_autoplaced yes)
-		(property "Reference" "#PWR027"
+		(property "Reference" "#PWR024"
 			(at 119.38 130.81 0)
 			(effects
@@
 			(project "RPi-HwAB-1"
 				(path "/e63e39d7-6ac0-4ffd-8aa3-1841a4541b55/59d21473-a004-4514-8090-fd93db818925/143e814b-c088-43b0-8f2f-ada8c438e494"
-					(reference "#PWR027")
+					(reference "#PWR024")
 					(unit 1)
 				)
@@
 		(dnp no)
 		(fields_autoplaced yes)
-		(property "Reference" "#PWR028"
+		(property "Reference" "#PWR026"
 			(at 71.12 194.31 0)
 			(effects
@@
 			(project "RPi-HwAB-1"
 				(path "/e63e39d7-6ac0-4ffd-8aa3-1841a4541b55/59d21473-a004-4514-8090-fd93db818925/143e814b-c088-43b0-8f2f-ada8c438e494"
-					(reference "#PWR028")
+					(reference "#PWR026")
 					(unit 1)
 				)
@@
 		(on_board yes)
 		(dnp no)
-		(property "Reference" "C32"
+		(property "Reference" "C31"
 			(at 227.33 138.43 0)
 			(effects
@@
 			(project "RPi-HwAB-1"
 				(path "/e63e39d7-6ac0-4ffd-8aa3-1841a4541b55/59d21473-a004-4514-8090-fd93db818925/143e814b-c088-43b0-8f2f-ada8c438e494"
-					(reference "C32")
+					(reference "C31")
 					(unit 1)
 				)
@@
 		(on_board yes)
 		(dnp no)
-		(property "Reference" "C33"
+		(property "Reference" "C32"
 			(at 234.95 138.43 0)
 			(effects
@@
 			(project "RPi-HwAB-1"
 				(path "/e63e39d7-6ac0-4ffd-8aa3-1841a4541b55/59d21473-a004-4514-8090-fd93db818925/143e814b-c088-43b0-8f2f-ada8c438e494"
-					(reference "C33")
+					(reference "C32")
 					(unit 1)
 				)
@@
 		(on_board yes)
 		(dnp no)
-		(property "Reference" "C30"
+		(property "Reference" "C29"
 			(at 110.49 119.38 0)
 			(effects
@@
 			(project "RPi-HwAB-1"
 				(path "/e63e39d7-6ac0-4ffd-8aa3-1841a4541b55/59d21473-a004-4514-8090-fd93db818925/143e814b-c088-43b0-8f2f-ada8c438e494"
-					(reference "C30")
+					(reference "C29")
 					(unit 1)
 				)
@@
 		(on_board yes)
 		(dnp no)
-		(property "Reference" "C34"
+		(property "Reference" "C33"
 			(at 242.57 138.43 0)
 			(effects
@@
 			(project "RPi-HwAB-1"
 				(path "/e63e39d7-6ac0-4ffd-8aa3-1841a4541b55/59d21473-a004-4514-8090-fd93db818925/143e814b-c088-43b0-8f2f-ada8c438e494"
-					(reference "C34")
+					(reference "C33")
 					(unit 1)
 				)
@@
 		(on_board yes)
 		(dnp no)
-		(property "Reference" "C35"
+		(property "Reference" "C34"
 			(at 250.19 138.43 0)
 			(effects
@@
 			(project "RPi-HwAB-1"
 				(path "/e63e39d7-6ac0-4ffd-8aa3-1841a4541b55/59d21473-a004-4514-8090-fd93db818925/143e814b-c088-43b0-8f2f-ada8c438e494"
-					(reference "C35")
+					(reference "C34")
 					(unit 1)
 				)
@@
 		(on_board yes)
 		(dnp no)
-		(property "Reference" "C29"
+		(property "Reference" "C28"
 			(at 102.87 119.38 0)
 			(effects
@@
 			(project "RPi-HwAB-1"
 				(path "/e63e39d7-6ac0-4ffd-8aa3-1841a4541b55/59d21473-a004-4514-8090-fd93db818925/143e814b-c088-43b0-8f2f-ada8c438e494"
-					(reference "C29")
+					(reference "C28")
 					(unit 1)
 				)

Commit message: length matched ddr upper and lower data bytes, pending address
Connections:
- net DQ0: now also U4.G2 (IO_L8N_T1_AD14N_35); no longer U4.H3 (IO_L11P_T1_SRCC_35)
- net DQ1: now also U4.G3 (IO_L11N_T1_SRCC_35); no longer U4.G2 (IO_L8N_T1_AD14N_35)
- net DQ2: now also U4.H2 (IO_L8P_T1_AD14P_35); no longer U4.H4 (IO_L12P_T1_MRCC_35)
- net DQ3: now also U4.H3 (IO_L11P_T1_SRCC_35); no longer U4.G3 (IO_L11N_T1_SRCC_35)
- net DQ5: now also U4.H5 (IO_L10N_T1_AD15N_35); no longer U4.J1 (IO_L7N_T1_AD6N_35)
- net DQ6: now also U4.H4 (IO_L12P_T1_MRCC_35); no longer U4.H5 (IO_L10N_T1_AD15N_35)
- net DQ7: now also U4.J1 (IO_L7N_T1_AD6N_35); no longer U4.H2 (IO_L8P_T1_AD14P_35)
Changed lines of the file:
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@@
 	)
 	(label "DQ6"
-		(at 198.12 76.2 180)
+		(at 198.12 83.82 180)
 		(effects
 			(font
@@
 	)
 	(label "DQ7"
-		(at 198.12 63.5 180)
+		(at 198.12 60.96 180)
 		(effects
 			(font
@@
 	)
 	(label "DQ0"
-		(at 198.12 78.74 180)
+		(at 198.12 66.04 180)
 		(effects
 			(font
@@
 	)
 	(label "DQ1"
-		(at 198.12 66.04 180)
+		(at 198.12 81.28 180)
 		(effects
 			(font
@@
 	)
 	(label "DQ3"
-		(at 198.12 81.28 180)
+		(at 198.12 78.74 180)
 		(effects
 			(font
@@
 	)
 	(label "DQ5"
-		(at 198.12 60.96 180)
+		(at 198.12 76.2 180)
 		(effects
 			(font
@@
 	)
 	(label "DQ2"
-		(at 198.12 83.82 180)
-		(effects
-			(font
+		(at 198.12 63.5 180)
+		(effects
+			(font
