File: pcb/sensors.kicad_sch (KiCad schematic)
At the start: 10 parts, among them U10 INA230AIRGTT, U11 MCP9804_DFN, U7 INA230AIRGTT, U9 INA230AIRGTT

Commit message: moved stuff around, bom
Parts:
- renumbered C103 to C105, C104 to C106, C105 to C107, C106 to C108, U9 to U11, U7 to U12, U10 to U13, U11 to U14
Changed lines of the file:
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@@
 		(on_board yes)
 		(dnp no)
-		(property "Reference" "C106"
+		(property "Reference" "C108"
 			(at 186.69 86.3599 0)
 			(effects
@@
 			(project "RPi-HwAB-1"
 				(path "/e63e39d7-6ac0-4ffd-8aa3-1841a4541b55/010325a2-ae86-4ae0-96e8-1d16e8e45471"
-					(reference "C106")
+					(reference "C108")
 					(unit 1)
 				)
@@
 		(dnp no)
 		(fields_autoplaced yes)
-		(property "Reference" "C104"
+		(property "Reference" "C106"
 			(at 133.35 129.5399 0)
 			(effects
@@
 			(project "RPi-HwAB-1"
 				(path "/e63e39d7-6ac0-4ffd-8aa3-1841a4541b55/010325a2-ae86-4ae0-96e8-1d16e8e45471"
-					(reference "C104")
+					(reference "C106")
 					(unit 1)
 				)
@@
 		(dnp no)
 		(fields_autoplaced yes)
-		(property "Reference" "C105"
+		(property "Reference" "C107"
 			(at 133.35 180.3399 0)
 			(effects
@@
 			(project "RPi-HwAB-1"
 				(path "/e63e39d7-6ac0-4ffd-8aa3-1841a4541b55/010325a2-ae86-4ae0-96e8-1d16e8e45471"
-					(reference "C105")
+					(reference "C107")
 					(unit 1)
 				)
@@
 		(dnp no)
 		(fields_autoplaced yes)
-		(property "Reference" "#PWR042"
+		(property "Reference" "#PWR035"
 			(at 83.82 194.31 0)
 			(effects
@@
 			(project "RPi-HwAB-1"
 				(path "/e63e39d7-6ac0-4ffd-8aa3-1841a4541b55/010325a2-ae86-4ae0-96e8-1d16e8e45471"
-					(reference "#PWR042")
+					(reference "#PWR035")
 					(unit 1)
 				)
@@
 		(dnp no)
 		(fields_autoplaced yes)
-		(property "Reference" "U10"
+		(property "Reference" "U13"
 			(at 101.6 142.24 0)
 			(effects
@@
 			(project "RPi-HwAB-1"
 				(path "/e63e39d7-6ac0-4ffd-8aa3-1841a4541b55/010325a2-ae86-4ae0-96e8-1d16e8e45471"
-					(reference "U10")
+					(reference "U13")
 					(unit 1)
 				)
@@
 		(dnp no)
 		(fields_autoplaced yes)
-		(property "Reference" "#PWR026"
+		(property "Reference" "#PWR033"
 			(at 83.82 92.71 0)
 			(effects
@@
 			(project "RPi-HwAB-1"
 				(path "/e63e39d7-6ac0-4ffd-8aa3-1841a4541b55/010325a2-ae86-4ae0-96e8-1d16e8e45471"
-					(reference "#PWR026")
+					(reference "#PWR033")
 					(unit 1)
 				)
@@
 		(dnp no)
 		(fields_autoplaced yes)
-		(property "Reference" "#PWR044"
+		(property "Reference" "#PWR034"
 			(at 83.82 143.51 0)
 			(effects
@@
 			(project "RPi-HwAB-1"
 				(path "/e63e39d7-6ac0-4ffd-8aa3-1841a4541b55/010325a2-ae86-4ae0-96e8-1d16e8e45471"
-					(reference "#PWR044")
+					(reference "#PWR034")
 					(unit 1)
 				)
@@
 		(dnp no)
 		(fields_autoplaced yes)
-		(property "Reference" "C103"
+		(property "Reference" "C105"
 			(at 133.35 78.7399 0)
 			(effects
@@
 			(project ""
 				(path "/e63e39d7-6ac0-4ffd-8aa3-1841a4541b55/010325a2-ae86-4ae0-96e8-1d16e8e45471"
-					(reference "C103")
+					(reference "C105")
 					(unit 1)
 				)
@@
 		(on_board yes)
 		(dnp no)
-		(property "Reference" "U11"
+		(property "Reference" "U14"
 			(at 213.36 58.42 0)
 			(effects
@@
 			(project "RPi-HwAB-1"
 				(path "/e63e39d7-6ac0-4ffd-8aa3-1841a4541b55/010325a2-ae86-4ae0-96e8-1d16e8e45471"
-					(reference "U11")
+					(reference "U14")
 					(unit 1)
 				)
@@
 		(dnp no)
 		(fields_autoplaced yes)
-		(property "Reference" "#PWR028"
+		(property "Reference" "#PWR043"
 			(at 229.87 91.44 0)
 			(effects
@@
 			(project "RPi-HwAB-1"
 				(path "/e63e39d7-6ac0-4ffd-8aa3-1841a4541b55/010325a2-ae86-4ae0-96e8-1d16e8e45471"
-					(reference "#PWR028")
+					(reference "#PWR043")
 					(unit 1)
 				)
@@
 		(dnp no)
 		(fields_autoplaced yes)
-		(property "Reference" "#PWR029"
+		(property "Reference" "#PWR039"
 			(at 129.54 92.71 0)
 			(effects
@@
 			(project "RPi-HwAB-1"
 				(path "/e63e39d7-6ac0-4ffd-8aa3-1841a4541b55/010325a2-ae86-4ae0-96e8-1d16e8e45471"
-					(reference "#PWR029")
+					(reference "#PWR039")
 					(unit 1)
 				)
@@
 		(dnp no)
 		(fields_autoplaced yes)
-		(property "Reference" "#PWR047"
+		(property "Reference" "#PWR042"
 			(at 190.5 100.33 0)
 			(effects
@@
 			(project "RPi-HwAB-1"
 				(path "/e63e39d7-6ac0-4ffd-8aa3-1841a4541b55/010325a2-ae86-4ae0-96e8-1d16e8e45471"
-					(reference "#PWR047")
+					(reference "#PWR042")
 					(unit 1)
 				)
@@
 		(dnp no)
 		(fields_autoplaced yes)
-		(property "Reference" "#PWR027"
+		(property "Reference" "#PWR036"
 			(at 119.38 92.71 0)
 			(effects
@@
 			(project "RPi-HwAB-1"
 				(path "/e63e39d7-6ac0-4ffd-8aa3-1841a4541b55/010325a2-ae86-4ae0-96e8-1d16e8e45471"
-					(reference "#PWR027")
+					(reference "#PWR036")
 					(unit 1)
 				)
@@
 		(dnp no)
 		(fields_autoplaced yes)
-		(property "Reference" "#PWR043"
+		(property "Reference" "#PWR038"
 			(at 119.38 194.31 0)
 			(effects
@@
 			(project "RPi-HwAB-1"
 				(path "/e63e39d7-6ac0-4ffd-8aa3-1841a4541b55/010325a2-ae86-4ae0-96e8-1d16e8e45471"
-					(reference "#PWR043")
+					(reference "#PWR038")
 					(unit 1)
 				)
@@
 		(dnp no)
 		(fields_autoplaced yes)
-		(property "Reference" "#PWR045"
+		(property "Reference" "#PWR037"
 			(at 119.38 143.51 0)
 			(effects
@@
 			(project "RPi-HwAB-1"
 				(path "/e63e39d7-6ac0-4ffd-8aa3-1841a4541b55/010325a2-ae86-4ae0-96e8-1d16e8e45471"
-					(reference "#PWR045")
+					(reference "#PWR037")
 					(unit 1)
 				)
@@
 		(dnp no)
 		(fields_autoplaced yes)
-		(property "Reference" "U7"
+		(property "Reference" "U12"
 			(at 101.6 91.44 0)
 			(effects
@@
 			(project "RPi-HwAB-1"
 				(path "/e63e39d7-6ac0-4ffd-8aa3-1841a4541b55/010325a2-ae86-4ae0-96e8-1d16e8e45471"
-					(reference "U7")
+					(reference "U12")
 					(unit 1)
 				)
@@
 		(dnp no)
 		(fields_autoplaced yes)
-		(property "Reference" "U9"
+		(property "Reference" "U11"
 			(at 101.6 40.64 0)
 			(effects
@@
 			(project "RPi-HwAB-1"
 				(path "/e63e39d7-6ac0-4ffd-8aa3-1841a4541b55/010325a2-ae86-4ae0-96e8-1d16e8e45471"
-					(reference "U9")
+					(reference "U11")
 					(unit 1)
 				)
@@
 		(dnp no)
 		(fields_autoplaced yes)
-		(property "Reference" "#PWR046"
+		(property "Reference" "#PWR041"
 			(at 129.54 194.31 0)
 			(effects
@@
 			(project "RPi-HwAB-1"
 				(path "/e63e39d7-6ac0-4ffd-8aa3-1841a4541b55/010325a2-ae86-4ae0-96e8-1d16e8e45471"
-					(reference "#PWR046")
+					(reference "#PWR041")
 					(unit 1)
 				)
@@
 		(dnp no)
 		(fields_autoplaced yes)
-		(property "Reference" "#PWR030"
+		(property "Reference" "#PWR040"
 			(at 129.54 143.51 0)
 			(effects
@@
 			(project "RPi-HwAB-1"
 				(path "/e63e39d7-6ac0-4ffd-8aa3-1841a4541b55/010325a2-ae86-4ae0-96e8-1d16e8e45471"
-					(reference "#PWR030")
-					(unit 1)
-				)
+					(reference "#PWR040")
+					(unit 1)
+				)

Commit message: bom
Parts:
- C105, C106, C107, C108: Manufacturer (none) -> KEMET; Manufacturer Product Number (none) -> C0402C104K4RACTU; Part Description (none) -> CAP CER 0.1UF 16V X7R 0402
- R27: renamed from R25; Manufacturer (none) -> Vishay Dale; Manufacturer Product Number (none) -> CRCW04024K70FKED; Part Description (none) -> RES 4.7K OHM 1% 1/16W 0402
- R28: renamed from R26; Manufacturer (none) -> Vishay Dale; Manufacturer Product Number (none) -> CRCW04024K70FKED; Part Description (none) -> RES 4.7K OHM 1% 1/16W 0402
- U11, U12, U13: value INA230AIRGTT -> INA230AIRGTR; Manufacturer (none) -> Texas Instruments; Manufacturer Product Number (none) -> INA230AIRGTR; Part Description (none) -> IC CURRENT MONITOR 0.005 16VQFN
- U14: value MCP9804_DFN -> MCP9804T-E/MC; Manufacturer (none) -> Microchip Technology; Manufacturer Product Number (none) -> MCP9804T-E/MC; Part Description (none) -> SENSOR DIGITAL -40C-125C 8DFN
Connections:
- net 3V3 renamed 3V3_RPi

Commit message: added mig ddr pinout constraints
Parts:
- renumbered C105 to C67, C108 to C68, C106 to C69, C107 to C70, U14 to U12, U12 to U13, U13 to U14
Connections:
- net 3V3_RPi: now also U14.1 (A1); no longer U14.2 (A0)
- net GND: now also U14.2 (A0); no longer U14.1 (A1)
Other:
- note added: "ADDR: 0b1000010x 0x42 7bit"
Changed lines of the file:
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@@
 		)
 	)
-	(text "ADDR: 0b1000001x\n0x41 7bit"
+	(text "ADDR: 0b1000010x\n0x42 7bit"
 		(exclude_from_sim no)
 		(at 101.6 180.34 0)
@@
 	)
 	(junction
-		(at 152.4 160.02)
+		(at 152.4 157.48)
 		(diameter 0)
 		(color 0 0 255 1)
@@
 	)
 	(junction
+		(at 119.38 165.1)
+		(diameter 0)
+		(color 0 0 0 0)
+	)
+	(junction
 		(at 119.38 63.5)
 		(diameter 0)
@@
 	)
 	(junction
-		(at 119.38 165.1)
-		(diameter 0)
-		(color 0 0 0 0)
-	)
-	(junction
 		(at 229.87 71.12)
 		(diameter 0)
@@
 	(wire
 		(pts
-			(xy 119.38 157.48) (xy 119.38 165.1)
-		)
-		(stroke
-			(width 0)
-			(type default)
-		)
-	)
-	(wire
-		(pts
 			(xy 119.38 116.84) (xy 119.38 114.3)
 		)
@@
 	(wire
 		(pts
+			(xy 119.38 160.02) (xy 119.38 165.1)
+		)
+		(stroke
+			(width 0)
+			(type default)
+		)
+	)
+	(wire
+		(pts
 			(xy 152.4 109.22) (xy 152.4 124.46)
 		)
@@
 	(wire
 		(pts
-			(xy 116.84 160.02) (xy 152.4 160.02)
+			(xy 116.84 157.48) (xy 152.4 157.48)
 		)
 		(stroke
@@
 	(wire
 		(pts
-			(xy 116.84 157.48) (xy 119.38 157.48)
-		)
-		(stroke
-			(width 0)
-			(type default)
-		)
-	)
-	(wire
-		(pts
 			(xy 128.27 29.21) (xy 128.27 33.02)
 		)
@@
 	(wire
 		(pts
-			(xy 152.4 160.02) (xy 152.4 175.26)
+			(xy 116.84 160.02) (xy 119.38 160.02)
+		)
+		(stroke
+			(width 0)
+			(type default)
+		)
+	)
+	(wire
+		(pts
+			(xy 152.4 157.48) (xy 152.4 175.26)
 		)
 		(stroke
@@
 	(wire
 		(pts
-			(xy 152.4 124.46) (xy 152.4 160.02)
+			(xy 152.4 124.46) (xy 152.4 157.48)
 		)
 		(stroke
@@
 		)
 	)
+	(label "3V3_RPi"
+		(at 43.18 17.78 0)
+		(effects
+			(font
+				(size 1.27 1.27)
+			)
+			(justify left bottom)
+		)
+	)
 	(label "I2C1.SCL"
 		(at 58.42 33.02 0)
@@
 		(on_board yes)
 		(dnp no)
-		(property "Reference" "C108"
+		(property "Reference" "C68"
 			(at 186.69 86.3599 0)
 			(effects
@@
 			(project "RPi-HwAB-1"
 				(path "/e63e39d7-6ac0-4ffd-8aa3-1841a4541b55/010325a2-ae86-4ae0-96e8-1d16e8e45471"
-					(reference "C108")
+					(reference "C68")
 					(unit 1)
 				)
@@
 		(dnp no)
 		(fields_autoplaced yes)
-		(property "Reference" "C106"
+		(property "Reference" "C69"
 			(at 133.35 129.5399 0)
 			(effects
@@
 			(project "RPi-HwAB-1"
 				(path "/e63e39d7-6ac0-4ffd-8aa3-1841a4541b55/010325a2-ae86-4ae0-96e8-1d16e8e45471"
-					(reference "C106")
+					(reference "C69")
 					(unit 1)
 				)
@@
 		(dnp no)
 		(fields_autoplaced yes)
-		(property "Reference" "C107"
+		(property "Reference" "C70"
 			(at 133.35 180.3399 0)
 			(effects
@@
 			(project "RPi-HwAB-1"
 				(path "/e63e39d7-6ac0-4ffd-8aa3-1841a4541b55/010325a2-ae86-4ae0-96e8-1d16e8e45471"
-					(reference "C107")
+					(reference "C70")
 					(unit 1)
 				)
@@
 		(dnp no)
 		(fields_autoplaced yes)
-		(property "Reference" "#PWR053"
+		(property "Reference" "#PWR055"
 			(at 83.82 194.31 0)
 			(effects
@@
 			(project "RPi-HwAB-1"
 				(path "/e63e39d7-6ac0-4ffd-8aa3-1841a4541b55/010325a2-ae86-4ae0-96e8-1d16e8e45471"
-					(reference "#PWR053")
+					(reference "#PWR055")
 					(unit 1)
 				)
@@
 		(dnp no)
 		(fields_autoplaced yes)
-		(property "Reference" "U13"
+		(property "Reference" "U14"
 			(at 101.6 142.24 0)
 			(effects
@@
 			(project "RPi-HwAB-1"
 				(path "/e63e39d7-6ac0-4ffd-8aa3-1841a4541b55/010325a2-ae86-4ae0-96e8-1d16e8e45471"
-					(reference "U13")
+					(reference "U14")
 					(unit 1)
 				)
@@
 		(dnp no)
 		(fields_autoplaced yes)
-		(property "Reference" "#PWR051"
+		(property "Reference" "#PWR048"
 			(at 83.82 92.71 0)
 			(effects
@@
 			(project "RPi-HwAB-1"
 				(path "/e63e39d7-6ac0-4ffd-8aa3-1841a4541b55/010325a2-ae86-4ae0-96e8-1d16e8e45471"
-					(reference "#PWR051")
+					(reference "#PWR048")
 					(unit 1)
 				)
@@
 		(dnp no)
 		(fields_autoplaced yes)
-		(property "Reference" "C105"
+		(property "Reference" "C67"
 			(at 133.35 78.7399 0)
 			(effects
@@
 			(project ""
 				(path "/e63e39d7-6ac0-4ffd-8aa3-1841a4541b55/010325a2-ae86-4ae0-96e8-1d16e8e45471"
-					(reference "C105")
+					(reference "C67")
 					(unit 1)
 				)
@@
 		(on_board yes)
 		(dnp no)
-		(property "Reference" "U14"
+		(property "Reference" "U12"
 			(at 213.36 58.42 0)
 			(effects
@@
 			(project "RPi-HwAB-1"
 				(path "/e63e39d7-6ac0-4ffd-8aa3-1841a4541b55/010325a2-ae86-4ae0-96e8-1d16e8e45471"
-					(reference "U14")
+					(reference "U12")
 					(unit 1)
 				)
@@
 		(dnp no)
 		(fields_autoplaced yes)
-		(property "Reference" "#PWR061"
+		(property "Reference" "#PWR047"
 			(at 229.87 91.44 0)
 			(effects
@@
 			(project "RPi-HwAB-1"
 				(path "/e63e39d7-6ac0-4ffd-8aa3-1841a4541b55/010325a2-ae86-4ae0-96e8-1d16e8e45471"
-					(reference "#PWR061")
+					(reference "#PWR047")
 					(unit 1)
 				)
@@
 		(dnp no)
 		(fields_autoplaced yes)
-		(property "Reference" "#PWR057"
+		(property "Reference" "#PWR050"
 			(at 129.54 92.71 0)
 			(effects
@@
 			(project "RPi-HwAB-1"
 				(path "/e63e39d7-6ac0-4ffd-8aa3-1841a4541b55/010325a2-ae86-4ae0-96e8-1d16e8e45471"
-					(reference "#PWR057")
+					(reference "#PWR050")
 					(unit 1)
 				)
@@
 		(dnp no)
 		(fields_autoplaced yes)
-		(property "Reference" "#PWR060"
+		(property "Reference" "#PWR051"
 			(at 190.5 100.33 0)
 			(effects
@@
 			(project "RPi-HwAB-1"
 				(path "/e63e39d7-6ac0-4ffd-8aa3-1841a4541b55/010325a2-ae86-4ae0-96e8-1d16e8e45471"
-					(reference "#PWR060")
+					(reference "#PWR051")
 					(unit 1)
 				)
@@
 		(dnp no)
 		(fields_autoplaced yes)
-		(property "Reference" "#PWR054"
+		(property "Reference" "#PWR049"
 			(at 119.38 92.71 0)
 			(effects
@@
 			(project "RPi-HwAB-1"
 				(path "/e63e39d7-6ac0-4ffd-8aa3-1841a4541b55/010325a2-ae86-4ae0-96e8-1d16e8e45471"
-					(reference "#PWR054")
+					(reference "#PWR049")
 					(unit 1)
 				)
@@
 		(dnp no)
 		(fields_autoplaced yes)
-		(property "Reference" "#PWR055"
+		(property "Reference" "#PWR053"
 			(at 119.38 143.51 0)
 			(effects
@@
 			(project "RPi-HwAB-1"
 				(path "/e63e39d7-6ac0-4ffd-8aa3-1841a4541b55/010325a2-ae86-4ae0-96e8-1d16e8e45471"
-					(reference "#PWR055")
+					(reference "#PWR053")
 					(unit 1)
 				)
@@
 		(dnp no)
 		(fields_autoplaced yes)
-		(property "Reference" "U12"
+		(property "Reference" "U13"
 			(at 101.6 91.44 0)
 			(effects
@@
 			(project "RPi-HwAB-1"
 				(path "/e63e39d7-6ac0-4ffd-8aa3-1841a4541b55/010325a2-ae86-4ae0-96e8-1d16e8e45471"
-					(reference "U12")
+					(reference "U13")
 					(unit 1)
 				)
@@
 		(dnp no)
 		(fields_autoplaced yes)
-		(property "Reference" "#PWR059"
+		(property "Reference" "#PWR057"
 			(at 129.54 194.31 0)
 			(effects
@@
 			(project "RPi-HwAB-1"
 				(path "/e63e39d7-6ac0-4ffd-8aa3-1841a4541b55/010325a2-ae86-4ae0-96e8-1d16e8e45471"
-					(reference "#PWR059")
+					(reference "#PWR057")
 					(unit 1)
 				)
@@
 		(dnp no)
 		(fields_autoplaced yes)
-		(property "Reference" "#PWR058"
+		(property "Reference" "#PWR054"
 			(at 129.54 143.51 0)
 			(effects
@@
 			(project "RPi-HwAB-1"
 				(path "/e63e39d7-6ac0-4ffd-8aa3-1841a4541b55/010325a2-ae86-4ae0-96e8-1d16e8e45471"
-					(reference "#PWR058")
+					(reference "#PWR054")
 					(unit 1)
 				)
