File: pcb/fpga-4.kicad_sch (KiCad schematic)
At the start: 9 parts, among them U4 XC7A100T-FGG484

Commit message: added jlc fab
Parts:
- R19: Manufacturer Vishay Dale -> YAGEO; Manufacturer Product Number CRCW04021K00FKED -> RC0402JR-071KL; Part Description RES 1K OHM 1% 1/16W 0402 -> RES 1K OHM 5% 1/16W 0402
Changed lines of the file:
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@@
 			)
 		)
-		(property "Manufacturer" "Vishay Dale"
+		(property "Manufacturer" "YAGEO"
 			(at 147.32 135.89 0)
 			(hide yes)
@@
 			)
 		)
-		(property "Manufacturer Product Number" "CRCW04021K00FKED"
+		(property "Manufacturer Product Number" "RC0402JR-071KL"
 			(at 147.32 135.89 0)
 			(hide yes)
@@
 			)
 		)
-		(property "Part Description" "RES 1K OHM 1% 1/16W 0402"
+		(property "Part Description" "RES 1K OHM 5% 1/16W 0402"
 			(at 147.32 135.89 0)
 			(hide yes)
